Commit message: 删除Taks_T1.csv文件并更新URDF网格路径
- 删除assets/Taks_T1/urdf/Taks_T1.csv文件(包含14行机器人链接参数数据)
- 修改Taks_T1.urdf中所有网格文件路径,从"meshes/"改为"../meshes/"
- 涉及所有机器人部件的visual和collision几何体定义,包括骨盆、髋关节、膝关节、踝关节、腰部、肩部、肘部和腕部链接

File: assets/Taks_T1/urdf/Taks_T1.urdf (robot description, URDF)
Before this commit: robot Taks_T1, 33 links, 32 joints
Links:
- added link head_mocap
- link left_ankle_pitch_link: geometry collision mesh filename=../meshes/left_ankle_pitch_link.STL; visual mesh filename=../meshes/left_ankle_pitch_link.STL
- link left_ankle_roll_link: geometry collision mesh filename=../meshes/left_ankle_roll_link.STL; visual mesh filename=../meshes/left_ankle_roll_link.STL
- link left_elbow_link: geometry collision mesh filename=../meshes/left_elbow_link.STL; visual mesh filename=../meshes/left_elbow_link.STL
- link left_hip_pitch_link: geometry collision mesh filename=../meshes/left_hip_pitch_link.STL; visual mesh filename=../meshes/left_hip_pitch_link.STL
- link left_hip_roll_link: geometry collision mesh filename=../meshes/left_hip_roll_link.STL; visual mesh filename=../meshes/left_hip_roll_link.STL
- link left_hip_yaw_link: geometry collision mesh filename=../meshes/left_hip_yaw_link.STL; visual mesh filename=../meshes/left_hip_yaw_link.STL
- link left_knee_link: geometry collision mesh filename=../meshes/left_knee_link.STL; visual mesh filename=../meshes/left_knee_link.STL
- link left_shoulder_pitch_link: geometry collision mesh filename=../meshes/left_shoulder_pitch_link.STL; visual mesh filename=../meshes/left_shoulder_pitch_link.STL
- link left_shoulder_roll_link: geometry collision mesh filename=../meshes/left_shoulder_roll_link.STL; visual mesh filename=../meshes/left_shoulder_roll_link.STL
- link left_shoulder_yaw_link: geometry collision mesh filename=../meshes/left_shoulder_yaw_link.STL; visual mesh filename=../meshes/left_shoulder_yaw_link.STL
- link left_wrist_pitch_link: geometry collision mesh filename=../meshes/left_wrist_pitch_link.STL; visual mesh filename=../meshes/left_wrist_pitch_link.STL
- link left_wrist_roll_link: geometry collision mesh filename=../meshes/left_wrist_roll_link.STL; visual mesh filename=../meshes/left_wrist_roll_link.STL
- link left_wrist_yaw_link: geometry collision mesh filename=../meshes/left_wrist_yaw_link.STL; visual mesh filename=../meshes/left_wrist_yaw_link.STL
- link neck_pitch_link: geometry collision mesh filename=../meshes/neck_pitch_link.STL; visual mesh filename=../meshes/neck_pitch_link.STL
- link neck_roll_link: geometry collision mesh filename=../meshes/neck_roll_link.STL; visual mesh filename=../meshes/neck_roll_link.STL
- link neck_yaw_link: geometry collision mesh filename=../meshes/neck_yaw_link.STL; visual mesh filename=../meshes/neck_yaw_link.STL
- link pelvis: geometry collision mesh filename=../meshes/pelvis.STL; visual mesh filename=../meshes/pelvis.STL
- link right_ankle_pitch_link: geometry collision mesh filename=../meshes/right_ankle_pitch_link.STL; visual mesh filename=../meshes/right_ankle_pitch_link.STL
- link right_ankle_roll_link: geometry collision mesh filename=../meshes/right_ankle_roll_link.STL; visual mesh filename=../meshes/right_ankle_roll_link.STL
- link right_elbow_link: geometry collision mesh filename=../meshes/right_elbow_link.STL; visual mesh filename=../meshes/right_elbow_link.STL
- link right_hip_pitch_link: geometry collision mesh filename=../meshes/right_hip_pitch_link.STL; visual mesh filename=../meshes/right_hip_pitch_link.STL
- link right_hip_roll_link: geometry collision mesh filename=../meshes/right_hip_roll_link.STL; visual mesh filename=../meshes/right_hip_roll_link.STL
- link right_hip_yaw_link: geometry collision mesh filename=../meshes/right_hip_yaw_link.STL; visual mesh filename=../meshes/right_hip_yaw_link.STL
- link right_knee_link: geometry collision mesh filename=../meshes/right_knee_link.STL; visual mesh filename=../meshes/right_knee_link.STL
- link right_shoulder_pitch_link: geometry collision mesh filename=../meshes/right_shoulder_pitch_link.STL; visual mesh filename=../meshes/right_shoulder_pitch_link.STL
- link right_shoulder_roll_link: geometry collision mesh filename=../meshes/right_shoulder_roll_link.STL; visual mesh filename=../meshes/right_shoulder_roll_link.STL
- link right_shoulder_yaw_link: geometry collision mesh filename=../meshes/right_shoulder_yaw_link.STL; visual mesh filename=../meshes/right_shoulder_yaw_link.STL
- link right_wrist_pitch_link: geometry collision mesh filename=../meshes/right_wrist_pitch_link.STL; visual mesh filename=../meshes/right_wrist_pitch_link.STL
- link right_wrist_roll_link: geometry collision mesh filename=../meshes/right_wrist_roll_link.STL; visual mesh filename=../meshes/right_wrist_roll_link.STL
- link right_wrist_yaw_link: geometry collision mesh filename=../meshes/right_wrist_yaw_link.STL; visual mesh filename=../meshes/right_wrist_yaw_link.STL
- link torso_link: geometry collision mesh filename=../meshes/waist_pitch_link.STL; visual mesh filename=../meshes/waist_pitch_link.STL
- link waist_roll_link: geometry collision mesh filename=../meshes/waist_roll_link.STL; visual mesh filename=../meshes/waist_roll_link.STL
- link waist_yaw_link: geometry collision mesh filename=../meshes/waist_yaw_link.STL; visual mesh filename=../meshes/waist_yaw_link.STL
Joints:
- added joint head_mocap_joint: type fixed, parent torso_link, child head_mocap, origin xyz=0.0 0.032906 0.5 rpy=0 0 0

Commit message: 更新Taks_T1机器人URDF和MuJoCo配置文件
- 修改URDF中所有碰撞几何体从mesh改为capsule简化碰撞检测
- 为所有碰撞几何体添加详细的MuJoCo标签,包括名称、组别、碰撞类型(contype)和碰撞亲和性(conaffinity)参数
- 调整碰撞几何体的位置和方向以更好地匹配实际机器人形状
- 将网格文件路径从"../meshes/"改回"meshes/"
- 更新MuJoCo XML配置文件中的home关键帧姿态,将所有关节角度从非零值重置为0

File: assets/Taks_T1/urdf/Taks_T1.urdf (robot description, URDF)
Before this commit: robot Taks_T1, 34 links, 33 joints
Links:
- removed link head_mocap
- link left_ankle_pitch_link: geometry collision capsule length=0.02 radius=0.015; visual mesh filename=meshes/left_ankle_pitch_link.STL
- link left_ankle_roll_link: geometry collision capsule length=0.14 radius=0.025; visual mesh filename=meshes/left_ankle_roll_link.STL
- link left_elbow_link: geometry collision capsule length=0.1 radius=0.03; visual mesh filename=meshes/left_elbow_link.STL
- link left_hip_pitch_link: geometry collision capsule length=0.06 radius=0.04; visual mesh filename=meshes/left_hip_pitch_link.STL
- link left_hip_roll_link: geometry collision capsule length=0.08 radius=0.04; visual mesh filename=meshes/left_hip_roll_link.STL
- link left_hip_yaw_link: geometry collision capsule length=0.2 radius=0.05; visual mesh filename=meshes/left_hip_yaw_link.STL
- link left_knee_link: geometry collision capsule length=0.24 radius=0.04; visual mesh filename=meshes/left_knee_link.STL
- link left_shoulder_pitch_link: geometry collision capsule length=0.05 radius=0.03; visual mesh filename=meshes/left_shoulder_pitch_link.STL
- link left_shoulder_roll_link: geometry collision capsule length=0.08 radius=0.035; visual mesh filename=meshes/left_shoulder_roll_link.STL
- link left_shoulder_yaw_link: geometry collision capsule length=0.14 radius=0.035; visual mesh filename=meshes/left_shoulder_yaw_link.STL
- link left_wrist_pitch_link: geometry collision capsule length=0.1 radius=0.025; visual mesh filename=meshes/left_wrist_pitch_link.STL
- link left_wrist_roll_link: geometry collision capsule length=0.1 radius=0.025; visual mesh filename=meshes/left_wrist_roll_link.STL
- link left_wrist_yaw_link: geometry collision capsule length=0.04 radius=0.02; visual mesh filename=meshes/left_wrist_yaw_link.STL
- link neck_pitch_link: geometry collision capsule length=0.08 radius=0.07; visual mesh filename=meshes/neck_pitch_link.STL
- link neck_roll_link: geometry collision capsule length=0.06 radius=0.015; visual mesh filename=meshes/neck_roll_link.STL
- link neck_yaw_link: geometry collision capsule length=0.06 radius=0.03; visual mesh filename=meshes/neck_yaw_link.STL
- link pelvis: geometry collision capsule length=0.12 radius=0.08; visual mesh filename=meshes/pelvis.STL
- link right_ankle_pitch_link: geometry collision capsule length=0.02 radius=0.015; visual mesh filename=meshes/right_ankle_pitch_link.STL
- link right_ankle_roll_link: geometry collision capsule length=0.14 radius=0.025; visual mesh filename=meshes/right_ankle_roll_link.STL
- link right_elbow_link: geometry collision capsule length=0.1 radius=0.03; visual mesh filename=meshes/right_elbow_link.STL
- link right_hip_pitch_link: geometry collision capsule length=0.06 radius=0.04; visual mesh filename=meshes/right_hip_pitch_link.STL
- link right_hip_roll_link: geometry collision capsule length=0.08 radius=0.04; visual mesh filename=meshes/right_hip_roll_link.STL
- link right_hip_yaw_link: geometry collision capsule length=0.2 radius=0.05; visual mesh filename=meshes/right_hip_yaw_link.STL
- link right_knee_link: geometry collision capsule length=0.24 radius=0.04; visual mesh filename=meshes/right_knee_link.STL
- link right_shoulder_pitch_link: geometry collision capsule length=0.05 radius=0.03; visual mesh filename=meshes/right_shoulder_pitch_link.STL
- link right_shoulder_roll_link: geometry collision capsule length=0.08 radius=0.035; visual mesh filename=meshes/right_shoulder_roll_link.STL
- link right_shoulder_yaw_link: geometry collision capsule length=0.14 radius=0.035; visual mesh filename=meshes/right_shoulder_yaw_link.STL
- link right_wrist_pitch_link: geometry collision capsule length=0.1 radius=0.025; visual mesh filename=meshes/right_wrist_pitch_link.STL
- link right_wrist_roll_link: geometry collision capsule length=0.1 radius=0.025; visual mesh filename=meshes/right_wrist_roll_link.STL
- link right_wrist_yaw_link: geometry collision capsule length=0.04 radius=0.02; visual mesh filename=meshes/right_wrist_yaw_link.STL
- link torso_link: geometry collision capsule length=0.08 radius=0.14; visual mesh filename=meshes/waist_pitch_link.STL
- link waist_roll_link: geometry collision capsule length=0.06 radius=0.06; visual mesh filename=meshes/waist_roll_link.STL
- link waist_yaw_link: geometry collision capsule length=0.04 radius=0.06; visual mesh filename=meshes/waist_yaw_link.STL
Joints:
- removed joint head_mocap_joint

Commit message: 为Taks_T1机器人URDF添加头部动作捕捉虚拟链接
- 在torso_link上添加head_mocap虚拟链接用于运动跟踪
- 使用固定关节连接,位置偏移为(0.0, 0.032906, 0.37165)
- 设置极小质量(0.001kg)和惯性参数以避免影响物理仿真

File: assets/Taks_T1/urdf/Taks_T1.urdf (robot description, URDF)
Before this commit: robot Taks_T1, 33 links, 32 joints
Links:
- added link head_mocap, mass 0.001
Joints:
- added joint head_mocap_joint: type fixed, parent torso_link, child head_mocap, origin xyz=0.0 0.032906 0.37165 rpy=0 0 0
